File: PCB/DSLogic_Breakout.kicad_sch (KiCad schematic)
At the start: 5 parts, among them J1 Interconnect

Commit message: Rev 1 Done
Parts:
- added D1: PWR, LED_SMD:LED_0603_1608Metric, symbol Device:LED
- added J2: Conn_Input, Connector_PinSocket_2.54mm:PinSocket_1x20_P2.54mm_Vertical, symbol Connector:Conn_01x20_Socket
- added R1: 2K2, Resistor_SMD:R_0603_1608Metric, symbol Device:R
Connections:
- net +3.3V: now also J2.1 (Pin_1), J2.2 (Pin_2), R1.1
- net GND: now also D1.1 (K), J2.19 (Pin_19), J2.20 (Pin_20)
- net INPUT_00: now also J2.3 (Pin_3)
- net INPUT_01: now also J2.4 (Pin_4)
- net INPUT_02: now also J2.5 (Pin_5)
- net INPUT_03: now also J2.6 (Pin_6)
- net INPUT_04: now also J2.7 (Pin_7)
- net INPUT_05: now also J2.8 (Pin_8)
- net INPUT_06: now also J2.9 (Pin_9)
- net INPUT_07: now also J2.10 (Pin_10)
- net INPUT_08: now also J2.11 (Pin_11)
- net INPUT_09: now also J2.12 (Pin_12)
- net INPUT_10: now also J2.13 (Pin_13)
- net INPUT_11: now also J2.14 (Pin_14)
- net INPUT_12: now also J2.15 (Pin_15)
- net INPUT_13: now also J2.16 (Pin_16)
- net INPUT_14: now also J2.17 (Pin_17)
- net INPUT_15: now also J2.18 (Pin_18)
- new net: D1.2 (A), R1.2
Other:
- title: (none) -> DSLogic Breakout
- moved on the sheet: J1, RN1, RN2, RN3, RN4
